File: Hardware/Mood-Badge.brd (EAGLE design)
At the start: 100 x 80 mm, 1 part, among them U1 328P

Commit message: Updated sch and brd
Parts:
- added C1, C2: 22p, LinnesLab-Passives:C0603
- added C3, C5: 0.1u, LinnesLab-Passives:C0603
- added C4: 2.2u, LinnesLab-Passives:C0603
- added C6, C9: 4.7u, LinnesLab-Passives:C0603
- added C7, C8: 1u, LinnesLab-Passives:C0603
- added D1, D2: (no value), LinnesLab-DiscreteSemi:USC
- added FTDI1: FTDI_DEVICE, LinnesLab-Connectors:FTDI_DEVICE
- added J1: AVR_SPI_PROG_3X2NS, LinnesLab-Connectors:2X3-NS
- added LDO1: MIC550X, LinnesLab-Power:SOT23-5
- added LED1: (no value), LinnesLab-LED:LED-0603
- added LED2: (no value), LinnesLab-Displays:DOTMATRIX_BL-M12A881UR
- added LIPO1: (no value), LinnesLab-Connectors:JST-2-SMD
- added R1: 10k, LinnesLab-Passives:R0603
- added R10, R11, R12, R13, R14, R2, R4, R5, R6, R7, R8, R9: (no value), LinnesLab-Passives:R0603
- added R3: 100k, LinnesLab-Passives:R0603
- added SW1, SW3, SW4, SW5: (no value), LinnesLab-Switches:SPST.KT11P4SM34LFS
- added SW2, SW6: SWITCH.JS202011JXQNUPWARDS, LinnesLab-Switches:SWITCH.00
- added U2: ATMEGA328P_TQFP, LinnesLab-Microcontrollers:TQFP32-08
- added USB1: USB.MICRO-BIGGERPADS, LinnesLab-Connectors:USB-MICRO-01.BIGGERPADS
- added Y1: 8MHz, LinnesLab-Clocks:CA-301
- U1: value 328P -> MCP73831.SOT23-5; device LinnesLab-Microcontrollers:DIP28 -> LinnesLab-Power:SOT23-5
- moved U1 80.3 mm to (-45.7, 40.6)
Connections:
- removed net N$14: U1.12
- removed net N$15: U1.13
- removed net N$16: U1.14
- removed net N$17: U1.15
- removed net N$18: U1.16
- removed net N$19: U1.17
- removed net N$20: U1.18
- removed net N$21: U1.19
- removed net N$5: U1.26
- new net 3.3V: C4.1, C5.1, C8.1, FTDI1.VCC, J1.2, LDO1.5, R1.2, SW3.1, SW3.2, SW4.1, SW4.2, SW5.1, SW5.2, SW6.1, U2.18, U2.4, U2.6
- new net ACTION: R14.2, SW5.3, SW5.4, U2.19
- new net CHRG.STAT: LED1.A, R3.1
- new net DTR: C3.1, FTDI1.DTR
- new net GND: C1.2, C2.2, C4.2, C5.2, C6.2, C7.2, C8.2, C9.2, FTDI1.CTS, FTDI1.GND, J1.6, LDO1.2, LIPO1.1, R12.1, R13.1, R14.1, R2.1, SW1.3, SW1.4, SW6.3, U1.2, U2.21, U2.3, U2.5, USB1.5, USB1.S1, USB1.S2, USB1.S3, USB1.S4, USB1.S5, USB1.S6
- new net LD1: R8.1, U2.2
- new net LD10: J1.1, LED2.10, U2.16
- new net LD11: J1.4, LED2.11, U2.15
- new net LD12: R7.1, U2.14
- new net LD13: LED2.13, U2.13
- new net LD14: R5.1, U2.12
- new net LD15: LED2.15, U2.11
- new net LD16: LED2.16, U2.10
- new net LD2: R10.1, U2.1
- new net LD3: LED2.3, U2.32
- new net LD4: LED2.4, U2.28
- new net LD5: R11.1, U2.27
- new net LD6: LED2.6, U2.26
- new net LD7: R9.1, U2.25
- new net LD8: R6.1, U2.24
- new net LD9: J1.3, R4.1, U2.17
- new net LEFT: R12.2, SW3.3, SW3.4, U2.23
- new net MODE: SW6.2, U2.9
- new net RESET: C3.2, J1.5, R1.1, SW1.1, SW1.2, U2.29
- new net RIGHT: R13.2, SW4.3, SW4.4, U2.22
- new net RXD: FTDI1.RXI, U2.30
- new net TXD: FTDI1.TXO, U2.31
- new net VIN: C7.1, C9.1, D1.-, D2.-, LDO1.1, LDO1.3, R3.2, U1.4
- new net VLIPO: C6.1, LIPO1.2, R2.2, SW2.2, U1.3, U1.5
- new net V_USB: D1.+, USB1.1
- net N$1: now also C2.1, U2.7, Y1.2; no longer U1.20, U1.21, U1.7
- net N$10: now also LED2.1, R8.2; no longer U1.4
- net N$11: now also LED2.7, R9.2; no longer U1.5
- net N$12: now also LED2.2, R10.2; no longer U1.6
- net N$13: now also LED2.5, R11.2; no longer U1.11
- net N$2: now also C1.1, U2.8, Y1.1; no longer U1.23
- net N$3: now also LED2.9, R4.2; no longer U1.24
- net N$4: now also D2.+, SW2.1; no longer U1.25
- net N$6: now also LED1.C, U1.1; no longer U1.27
- net N$7: now also LED2.14, R5.2; no longer U1.28
- net N$8: now also LED2.8, R6.2; no longer U1.2
- net N$9: now also LED2.12, R7.2; no longer U1.3

Commit message: updated
Parts:
- moved FTDI1 151.9 mm to (91.4, 1.27)
- moved LDO1 145.3 mm to (97.8, 58.4)
- moved U1 145.3 mm to (97.8, 63.5)
- moved D1 136.3 mm to (82.5, 48.3)
- moved R4 133.3 mm to (63.5, 44.5)
- moved R3 130.8 mm to (71.1, 62.2)
- moved R2 130.6 mm to (63.5, 39.4)
- moved USB1 129.4 mm to (96.5, 29.2), turned to 90 degrees
- moved LIPO1 123.0 mm to (80.0, 76.2)
- moved SW4 122.8 mm to (69.8, 3.81)
- moved R1 114.9 mm to (63.5, 25.4)
- moved SW5 114.7 mm to (49.5, 3.81)
- moved SW6 114.3 mm to (92.7, 72.4), turned to 270 degrees
- moved R12 113.1 mm to (71.1, 72.4)
- moved C4 111.1 mm to (35.6, 20.3)
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Connections:
- new net N$1: C3.2, R1.1, U2.29
- new net N$64: R2.2, U1.5
- net DTR: no longer C3.1
- net RESET: now also C3.1; no longer C3.2, R1.1, U2.29
- net VLIPO: no longer R2.2, U1.5

Commit message: hardware update
Parts:
- moved R12 86.9 mm to (17.8, 3.81)
- moved R14 72.2 mm to (58.4, 6.35), turned to 180 degrees
- moved R13 51.8 mm to (80.0, 6.35)
- turned U2 to 270 degrees
Routing:
- net 3.3V: track 0.00 -> 136.9 mm
- net GND: track 0.00 -> 72.3 mm
- net RIGHT: track 0.00 -> 7.92 mm
- net LEFT: track 0.00 -> 6.55 mm
- net ACTION: track 0.00 -> 6.31 mm

Commit message: Hardware update
Parts:
- moved USB1 93.7 mm to (6.35, 54.6)
- moved U1 89.5 mm to (8.89, 73.7)
- moved LDO1 88.0 mm to (10.2, 66.0)
- moved FTDI1 76.4 mm to (71.1, 74.9)
- moved SW6 76.2 mm to (16.5, 71.1)
- moved R9 71.6 mm to (92.7, 22.9)
- moved R4 69.7 mm to (5.08, 6.35), turned to 90 degrees
- moved SW5 69.3 mm to (39.4, 72.4)
- moved D1 64.5 mm to (19.1, 59.7)
- moved LIPO1 58.5 mm to (21.6, 78.7)
- moved R3 57.2 mm to (14.0, 59.7)
- moved C7 47.4 mm to (24.1, 69.8)
- moved R11 46.7 mm to (88.9, 24.1)
- moved R10 46.2 mm to (66.0, 33.0)
- moved SW1 46.0 mm to (14.0, 12.7)
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Routing:
- net RESET: track 0.00 -> 132.1 mm
- net 3.3V: track 136.9 -> 46.8 mm
- net N$42: track 0.00 -> 89.5 mm
- net LD6: track 0.00 -> 79.8 mm
- net RXD: track 0.00 -> 71.7 mm
- net LD4: track 0.00 -> 69.4 mm
- net TXD: track 0.00 -> 69.4 mm
- net LD9: track 0.00 -> 51.1 mm
- net N$39: track 0.00 -> 46.7 mm
- net N$38: track 0.00 -> 38.6 mm
- net LD7: track 0.00 -> 38.1 mm
- net LD10: track 0.00 -> 37.3 mm
- net LD3: track 0.00 -> 36.2 mm
- net LD5: track 0.00 -> 34.3 mm
- net GND: track 72.3 -> 102.6 mm, vias 0 -> 1
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- added copper zone on layer 1, net 3.3V

Commit message: Hardware/Mood-badge.brd
Parts:
- moved Y1 104.1 mm to (99.1, 55.9)
- moved SW6 45.4 mm to (2.54, 27.9)
- moved R5 34.2 mm to (38.1, 43.2), turned to 90 degrees
- moved SW5 30.5 mm to (48.3, 43.2)
- moved FTDI1 21.9 mm to (92.7, 78.7)
- moved SW1 17.8 mm to (31.8, 11.4)
- moved LIPO1 16.7 mm to (5.08, 76.2)
- moved LED1 16.3 mm to (30.5, 78.7), turned to 180 degrees
- moved D1 15.7 mm to (3.81, 63.5)
- moved LED2 13.0 mm to (49.5, 63.5)
- moved U1 9.16 mm to (16.5, 68.6), turned to 90 degrees
- moved R4 7.73 mm to (6.35, 14.0)
- moved C6 7.73 mm to (2.54, 45.7), turned to 90 degrees
- moved SW2 5.68 mm to (2.54, 38.1)
- moved USB1 4.02 mm to (2.54, 55.9), turned to 270 degrees
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Routing:
- net GND: track 102.6 -> 254.1 mm, vias 1 -> 12
- net ACTION: track 2.97 -> 126.6 mm, vias 0 -> 4
- net RESET: track 132.1 -> 55.0 mm, vias 0 -> 2
- net LD11: track 24.5 -> 98.0 mm, vias 0 -> 1
- net N$44: track 0.00 -> 71.6 mm
- net LD10: track 37.3 -> 106.6 mm, vias 0 -> 1
- net N$4: track 0.00 -> 67.6 mm, vias 0 -> 2
- net N$3: track 12.6 -> 73.7 mm, vias 0 -> 3
- net VLIPO: track 0.00 -> 52.3 mm, vias 0 -> 4
- net VIN: track 0.00 -> 49.1 mm
- net CHRG.STAT: track 0.00 -> 48.6 mm, vias 0 -> 2
- net LD15: track 0.00 -> 47.0 mm, vias 0 -> 1
- net MODE: track 0.00 -> 41.5 mm, vias 0 -> 2
- net LD13: track 0.00 -> 41.4 mm, vias 0 -> 2
- net 3.3V: track 46.8 -> 11.1 mm, vias 0 -> 2
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- added copper zone on layer 16, net GND

Commit message: New BOM
Parts:
- R10, R11, R4, R5, R6, R7, R8, R9: value (none) -> 205
- R12, R13, R14: value (none) -> 10k
Changed lines of the file:
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@@
 <attribute name="VALUE" x="47.625" y="20.955" size="0.7112" layer="27"/>
 </element>
-<element name="R10" library="LinnesLab-Passives" package="R0603" package3d_urn="urn:adsk.eagle:package:15661944/2" value="" x="66.04" y="33.02" smashed="yes">
+<element name="R10" library="LinnesLab-Passives" package="R0603" package3d_urn="urn:adsk.eagle:package:15661944/2" value="205" x="66.04" y="33.02" smashed="yes">
 <attribute name="NAME" x="65.405" y="33.655" size="0.7112" layer="25"/>
 <attribute name="VALUE" x="65.405" y="31.115" size="0.7112" layer="27"/>
 </element>
-<element name="R11" library="LinnesLab-Passives" package="R0603" package3d_urn="urn:adsk.eagle:package:15661944/2" value="" x="88.9" y="24.13" smashed="yes">
+<element name="R11" library="LinnesLab-Passives" package="R0603" package3d_urn="urn:adsk.eagle:package:15661944/2" value="205" x="88.9" y="24.13" smashed="yes">
 <attribute name="NAME" x="88.265" y="24.765" size="0.7112" layer="25"/>
 <attribute name="VALUE" x="88.265" y="22.225" size="0.7112" layer="27"/>
 </element>
-<element name="R12" library="LinnesLab-Passives" package="R0603" package3d_urn="urn:adsk.eagle:package:15661944/2" value="" x="46.99" y="17.78" smashed="yes" rot="R90">
+<element name="R12" library="LinnesLab-Passives" package="R0603" package3d_urn="urn:adsk.eagle:package:15661944/2" value="10k" x="46.99" y="17.78" smashed="yes" rot="R90">
 <attribute name="NAME" x="46.355" y="17.145" size="0.7112" layer="25" rot="R90"/>
 <attribute name="VALUE" x="48.895" y="17.145" size="0.7112" layer="27" rot="R90"/>
 </element>
-<element name="R13" library="LinnesLab-Passives" package="R0603" package3d_urn="urn:adsk.eagle:package:15661944/2" value="" x="58.42" y="11.43" smashed="yes" rot="R270">
+<element name="R13" library="LinnesLab-Passives" package="R0603" package3d_urn="urn:adsk.eagle:package:15661944/2" value="10k" x="58.42" y="11.43" smashed="yes" rot="R270">
 <attribute name="NAME" x="61.595" y="9.525" size="0.7112" layer="25" rot="R270"/>
 <attribute name="VALUE" x="56.515" y="12.065" size="0.7112" layer="27" rot="R270"/>
 </element>
-<element name="R14" library="LinnesLab-Passives" package="R0603" package3d_urn="urn:adsk.eagle:package:15661944/2" value="" x="49.53" y="17.78" smashed="yes" rot="R90">
+<element name="R14" library="LinnesLab-Passives" package="R0603" package3d_urn="urn:adsk.eagle:package:15661944/2" value="10k" x="49.53" y="17.78" smashed="yes" rot="R90">
 <attribute name="NAME" x="47.625" y="17.145" size="0.7112" layer="25" rot="R90"/>
 <attribute name="VALUE" x="51.435" y="17.145" size="0.7112" layer="27" rot="R90"/>
@@
 <attribute name="VALUE" x="13.335" y="57.785" size="0.7112" layer="27"/>
 </element>
-<element name="R4" library="LinnesLab-Passives" package="R0603" package3d_urn="urn:adsk.eagle:package:15661944/2" value="" x="6.35" y="13.97" smashed="yes" rot="R90">
+<element name="R4" library="LinnesLab-Passives" package="R0603" package3d_urn="urn:adsk.eagle:package:15661944/2" value="205" x="6.35" y="13.97" smashed="yes" rot="R90">
 <attribute name="NAME" x="5.715" y="14.605" size="0.7112" layer="25" rot="R90"/>
 <attribute name="VALUE" x="8.255" y="13.335" size="0.7112" layer="27" rot="R90"/>
 </element>
-<element name="R5" library="LinnesLab-Passives" package="R0603" package3d_urn="urn:adsk.eagle:package:15661944/2" value="" x="38.1" y="43.18" smashed="yes" rot="R90">
+<element name="R5" library="LinnesLab-Passives" package="R0603" package3d_urn="urn:adsk.eagle:package:15661944/2" value="205" x="38.1" y="43.18" smashed="yes" rot="R90">
 <attribute name="NAME" x="37.465" y="42.545" size="0.7112" layer="25" rot="R90"/>
 <attribute name="VALUE" x="40.005" y="42.545" size="0.7112" layer="27" rot="R90"/>
 </element>
-<element name="R6" library="LinnesLab-Passives" package="R0603" package3d_urn="urn:adsk.eagle:package:15661944/2" value="" x="57.15" y="20.32" smashed="yes">
+<element name="R6" library="LinnesLab-Passives" package="R0603" package3d_urn="urn:adsk.eagle:package:15661944/2" value="205" x="57.15" y="20.32" smashed="yes">
 <attribute name="NAME" x="56.515" y="20.955" size="0.7112" layer="25"/>
 <attribute name="VALUE" x="56.515" y="18.415" size="0.7112" layer="27"/>
 </element>
-<element name="R7" library="LinnesLab-Passives" package="R0603" package3d_urn="urn:adsk.eagle:package:15661944/2" value="" x="27.94" y="49.53" smashed="yes">
+<element name="R7" library="LinnesLab-Passives" package="R0603" package3d_urn="urn:adsk.eagle:package:15661944/2" value="205" x="27.94" y="49.53" smashed="yes">
 <attribute name="NAME" x="27.305" y="50.165" size="0.7112" layer="25"/>
 <attribute name="VALUE" x="27.305" y="47.625" size="0.7112" layer="27"/>
 </element>
-<element name="R8" library="LinnesLab-Passives" package="R0603" package3d_urn="urn:adsk.eagle:package:15661944/2" value="" x="58.42" y="33.02" smashed="yes">
+<element name="R8" library="LinnesLab-Passives" package="R0603" package3d_urn="urn:adsk.eagle:package:15661944/2" value="205" x="58.42" y="33.02" smashed="yes">
 <attribute name="NAME" x="57.785" y="33.655" size="0.7112" layer="25"/>
 <attribute name="VALUE" x="57.785" y="31.115" size="0.7112" layer="27"/>
 </element>
-<element name="R9" library="LinnesLab-Passives" package="R0603" package3d_urn="urn:adsk.eagle:package:15661944/2" value="" x="92.71" y="22.86" smashed="yes">
+<element name="R9" library="LinnesLab-Passives" package="R0603" package3d_urn="urn:adsk.eagle:package:15661944/2" value="205" x="92.71" y="22.86" smashed="yes">
 <attribute name="NAME" x="92.075" y="23.495" size="0.7112" layer="25"/>
 <attribute name="VALUE" x="92.075" y="20.955" size="0.7112" layer="27"/>

Commit message: Changes
Parts:
- R2: value (none) -> 4.7k
- moved Y1 57.3 mm to (47.2, 31.4), turned to 0 degrees
- moved C2 7.90 mm to (48.9, 34.5)
- moved LED1 4.09 mm to (26.5, 77.9)
- moved C1 3.72 mm to (47.3, 34.5), turned to 90 degrees
- moved FTDI1 2.84 mm to (90.3, 77.2)
- moved J1 1.19 mm to (4.65, 3.38)
- moved SW4 1.10 mm to (50.6, 11.3)
- moved SW2 1.09 mm to (3.63, 38.2)
- moved SW6 0.97 mm to (3.51, 28.0)
- moved LIPO1 0.74 mm to (5.77, 76.5)
- moved USB1 0.27 mm to (2.79, 55.8)
Routing:
- net GND: track 254.1 -> 61.9 mm, vias 12 -> 18
- net N$3: track 73.7 -> 4.58 mm, vias 3 -> 0
- net N$4: track 67.6 -> 4.21 mm, vias 2 -> 0
- net VIN: track 49.1 -> 60.6 mm, vias 0 -> 2
- net 3.3V: track 11.1 -> 0.00 mm, vias 2 -> 0
- net VLIPO: track 52.3 -> 55.2 mm
- net N$6: track 18.9 -> 16.1 mm
- net TXD: track 74.1 -> 71.6 mm
- net RXD: track 76.3 -> 73.8 mm
- net LD11: track 98.0 -> 96.8 mm
- net LD10: track 106.6 -> 105.4 mm
- net RESET: track 55.0 -> 53.8 mm
- net N$60: track 13.6 -> 12.5 mm
- net RIGHT: track 33.5 -> 32.4 mm
- net MODE: track 41.5 -> 40.6 mm

Commit message: orlando made changes and ordered boards
Parts:
- C1, C2: value 22p -> 0.1u
- C3: value 0.1u -> 2.2u
- C4: value 2.2u -> 22p
- C5: value 0.1u -> 22p
- R2: value 4.7k -> 100k
- R3: value 100k -> 4.7k
- U1: value MCP73831.SOT23-5 -> ATMEGA328P_TQFP; device LinnesLab-Power:SOT23-5 -> LinnesLab-Microcontrollers:TQFP32-08
- U2: value ATMEGA328P_TQFP -> MCP73831.SOT23-5; device LinnesLab-Microcontrollers:TQFP32-08 -> LinnesLab-Power:SOT23-5
- moved U1 54.4 mm to (49.5, 25.4), turned to 270 degrees
- moved U2 54.4 mm to (16.5, 68.6), turned to 90 degrees
- moved C6 34.3 mm to (29.2, 67.3), turned to 0 degrees
- moved C9 34.3 mm to (2.54, 45.7), turned to 90 degrees
- moved SW5 32.0 mm to (50.6, 11.3)
- moved SW4 31.4 mm to (48.3, 42.5)
- moved C1 26.8 mm to (25.4, 19.1), turned to 270 degrees
- moved C5 26.8 mm to (47.3, 34.5), turned to 90 degrees
- moved R2 26.2 mm to (14.0, 59.7)
- moved R3 26.2 mm to (30.5, 39.4)
- moved C4 21.0 mm to (48.9, 34.5), turned to 90 degrees
- moved D1 18.1 mm to (15.2, 49.5)
- moved D2 18.1 mm to (3.81, 63.5)
- moved C3 14.5 mm to (40.6, 15.2), turned to 0 degrees
- moved C2 13.8 mm to (59.6, 25.8), turned to 180 degrees
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Connections:
- removed net N$1: C3.2, R1.1, U2.29
- net 3.3V: now also C1.1, C3.1, U1.18, U1.4, U1.6; no longer C4.1, C5.1, U2.18, U2.4, U2.6
- net ACTION: now also R13.2, SW4.3, SW4.4, U1.19; no longer R14.2, SW5.3, SW5.4, U2.19
- net CHRG.STAT: now also R2.1; no longer R3.1
- net DTR: now also C2.1
- net GND: now also C3.2, R3.1, U1.21, U1.3, U1.5, U2.2; no longer C2.2, R2.1, U1.2, U2.21, U2.3, U2.5
- net LD1: now also U1.2; no longer U2.2
- net LD10: now also U1.16; no longer U2.16
- net LD11: now also U1.15; no longer U2.15
- net LD12: now also U1.14; no longer U2.14
- net LD13: now also U1.13; no longer U2.13
- net LD14: now also U1.12; no longer U2.12
- net LD15: now also U1.11; no longer U2.11
- net LD16: now also U1.10; no longer U2.10
- net LD2: now also U1.1; no longer U2.1
- net LD3: now also U1.32; no longer U2.32
- net LD4: now also U1.28; no longer U2.28
- net LD5: now also U1.27; no longer U2.27
- net LD6: now also U1.26; no longer U2.26
- net LD7: now also U1.25; no longer U2.25
- net LD8: now also U1.24; no longer U2.24
- net LD9: now also U1.17; no longer U2.17
- net LEFT: now also U1.23; no longer U2.23
- net MODE: now also U1.9; no longer U2.9
- net N$3: now also C4.1, U1.7; no longer C2.1, U2.7
- net N$4: now also C5.1, U1.8; no longer C1.1, U2.8
- net N$6: now also U2.1; no longer U1.1
- net N$60: now also D1.+; no longer D2.+
- net N$64: now also R3.2, U2.5; no longer R2.2, U1.5
- net RESET: now also C2.2, R1.1, U1.29; no longer C3.1
- net RIGHT: now also R14.2, SW5.3, SW5.4, U1.22; no longer R13.2, SW4.3, SW4.4, U2.22
- net RXD: now also U1.30; no longer U2.30
- net TXD: now also U1.31; no longer U2.31
- net VIN: now also C6.1, R2.2, U2.4; no longer C9.1, R3.2, U1.4
- net VLIPO: now also C9.1, U2.3; no longer C6.1, U1.3
- net V_USB: now also D2.+; no longer D1.+
Routing:
- net DTR: track 0.00 -> 61.7 mm, vias 0 -> 2
- net N$1: track 32.2 -> 0.00 mm, vias 2 -> 1
- net RESET: track 53.8 -> 67.8 mm, vias 2 -> 3
- net GND: track 61.9 -> 70.6 mm, vias 18 -> 86
- net LD9: track 58.0 -> 55.4 mm
- net LD10: track 105.4 -> 103.3 mm
- net LD11: track 96.8 -> 94.7 mm, vias 1 -> 2
- net VIN: track 60.6 -> 58.6 mm
- net VLIPO: track 55.2 -> 53.5 mm
- net V_USB: track 7.61 -> 9.22 mm
- net TXD: track 71.6 -> 70.8 mm
- net RXD: track 73.8 -> 73.0 mm
