File: Hardware/Mood-Badge.sch (EAGLE design)
At the start: 7 parts, among them U2 ATMEGA328P_TQFP

Commit message: Updated sch and brd
Parts:
- added C6, C9: 4.7u, LinnesLab-Passives:CAPACITOR0603
- added C7, C8: 1u, LinnesLab-Passives:CAPACITOR0603
- added D1, D2: (no value), LinnesLab-DiscreteSemi:SCHOTTKY-USC
- added FTDI1: FTDI_DEVICE, LinnesLab-Connectors:FTDI_DEVICE
- added J1: AVR_SPI_PROG_3X2NS, LinnesLab-Connectors:AVR_SPI_PROG_3X2NS
- added LDO1: MIC550X, LinnesLab-Power:MIC550X
- added LED1: (no value), LinnesLab-LED:LED0603
- added LED2: (no value), LinnesLab-Displays:DOTMATRIX_8X8_ROWCATHODEM12A881UR
- added LIPO1: (no value), LinnesLab-Connectors:JST_2MM_MALE
- added R1: 10k, LinnesLab-Passives:RESISTOR0603
- added R10, R11, R12, R13, R14, R2, R4, R5, R6, R7, R8, R9: (no value), LinnesLab-Passives:RESISTOR0603
- added R3: 100k, LinnesLab-Passives:RESISTOR0603
- added SW1, SW3, SW4, SW5: (no value), LinnesLab-Switches:SPST.KT11P4SM34LFS
- added SW2, SW6: SWITCH.JS202011JXQNUPWARDS, LinnesLab-Switches:SWITCH.JS202011JXQNUPWARDS
- added U1: MCP73831.SOT23-5, LinnesLab-Power:MCP73831.SOT23-5
- added USB1: USB.MICRO-BIGGERPADS, LinnesLab-Connectors:USB.MICRO-BIGGERPADS
- C3, C5: value (none) -> 0.1u
- C4: value (none) -> 2.2u
- Y1: value (none) -> 8MHz
Connections:
- new net CHRG.STAT: LED1.A, R3.1
- new net DTR: C3.1, FTDI1.DTR
- new net N$10: LED2.K5, R8.2
- new net N$11: LED2.K6, R9.2
- new net N$12: LED2.K7, R10.2
- new net N$13: LED2.K8, R11.2
- new net N$3: LED2.K1, R4.2
- new net N$4: D2.A, SW2.1
- new net N$6: LED1.C, U1.STAT
- new net N$7: LED2.K2, R5.2
- new net N$8: LED2.K3, R6.2
- new net N$9: LED2.K4, R7.2
- new net RESET: C3.2, J1.5, R1.1, SW1.A, U2.PC6(/RESET)
- new net VIN: C7.1, C9.1, D1.C, D2.C, LDO1.EN, LDO1.IN, R3.2, U1.VIN
- new net VLIPO: C6.1, LIPO1.+, R2.2, SW2.2, U1.PROG, U1.VBAT
- new net V_USB: D1.A, USB1.V+
- net 3.3V: now also C8.1, FTDI1.VCC, J1.2, LDO1.OUT, R1.2, SW3.A, SW4.A, SW5.A, SW6.1, U2.AVCC, U2.VCC@4, U2.VCC@6
- net ACTION: now also R14.2, SW5.B
- net GND: now also C6.2, C7.2, C8.2, C9.2, FTDI1.CTS, FTDI1.GND, J1.6, LDO1.GND, LIPO1.-, R12.1, R13.1, R14.1, R2.1, SW1.B, SW6.3, U1.VSS, USB1.GND, USB1.SHIELD
- net LD1: now also R8.1
- net LD10: now also J1.1, LED2.A4
- net LD11: now also J1.4, LED2.A6
- net LD12: now also R7.1
- net LD13: now also LED2.A1
- net LD14: now also R5.1
- net LD15: now also LED2.A7
- net LD16: now also LED2.A8
- net LD2: now also R10.1
- net LD3: now also LED2.A2
- net LD4: now also LED2.A3
- net LD5: now also R11.1
- net LD6: now also LED2.A5
- net LD7: now also R9.1
- net LD8: now also R6.1
- net LD9: now also J1.3, R4.1
- net LEFT: now also R12.2, SW3.B
- net MODE: now also SW6.2
- net RIGHT: now also R13.2, SW4.B
- net RXD: now also FTDI1.TXO
- net TXD: now also FTDI1.RXI
Other:
- moved on the sheet: C3, C4, C5

Commit message: updated
Connections:
- new net N$1: C3.2, R1.1, U2.PC6(/RESET)
- new net N$64: R2.2, U1.PROG
- net DTR: no longer C3.1
- net RESET: now also C3.1; no longer C3.2, R1.1, U2.PC6(/RESET)
- net VLIPO: no longer R2.2, U1.PROG

Commit message: New BOM
Parts:
- R10, R11, R4, R5, R6, R7, R8, R9: value (none) -> 205
- R12, R13, R14: value (none) -> 10k
Changed lines of the file:
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@@
 <part name="GND16" library="LinnesLab-Symbols" deviceset="GND" device=""/>
 <part name="SUPPLY9" library="LinnesLab-Symbols" deviceset="3.3V" device=""/>
-<part name="R4" library="LinnesLab-Passives" deviceset="RESISTOR" device="0603" package3d_urn="urn:adsk.eagle:package:15661944/2"/>
-<part name="R5" library="LinnesLab-Passives" deviceset="RESISTOR" device="0603" package3d_urn="urn:adsk.eagle:package:15661944/2"/>
-<part name="R6" library="LinnesLab-Passives" deviceset="RESISTOR" device="0603" package3d_urn="urn:adsk.eagle:package:15661944/2"/>
-<part name="R7" library="LinnesLab-Passives" deviceset="RESISTOR" device="0603" package3d_urn="urn:adsk.eagle:package:15661944/2"/>
-<part name="R8" library="LinnesLab-Passives" deviceset="RESISTOR" device="0603" package3d_urn="urn:adsk.eagle:package:15661944/2"/>
-<part name="R9" library="LinnesLab-Passives" deviceset="RESISTOR" device="0603" package3d_urn="urn:adsk.eagle:package:15661944/2"/>
-<part name="R10" library="LinnesLab-Passives" deviceset="RESISTOR" device="0603" package3d_urn="urn:adsk.eagle:package:15661944/2"/>
-<part name="R11" library="LinnesLab-Passives" deviceset="RESISTOR" device="0603" package3d_urn="urn:adsk.eagle:package:15661944/2"/>
-<part name="R12" library="LinnesLab-Passives" deviceset="RESISTOR" device="0603" package3d_urn="urn:adsk.eagle:package:15661944/2"/>
-<part name="R13" library="LinnesLab-Passives" deviceset="RESISTOR" device="0603" package3d_urn="urn:adsk.eagle:package:15661944/2"/>
-<part name="R14" library="LinnesLab-Passives" deviceset="RESISTOR" device="0603" package3d_urn="urn:adsk.eagle:package:15661944/2"/>
+<part name="R4" library="LinnesLab-Passives" deviceset="RESISTOR" device="0603" package3d_urn="urn:adsk.eagle:package:15661944/2" value="205"/>
+<part name="R5" library="LinnesLab-Passives" deviceset="RESISTOR" device="0603" package3d_urn="urn:adsk.eagle:package:15661944/2" value="205"/>
+<part name="R6" library="LinnesLab-Passives" deviceset="RESISTOR" device="0603" package3d_urn="urn:adsk.eagle:package:15661944/2" value="205"/>
+<part name="R7" library="LinnesLab-Passives" deviceset="RESISTOR" device="0603" package3d_urn="urn:adsk.eagle:package:15661944/2" value="205"/>
+<part name="R8" library="LinnesLab-Passives" deviceset="RESISTOR" device="0603" package3d_urn="urn:adsk.eagle:package:15661944/2" value="205"/>
+<part name="R9" library="LinnesLab-Passives" deviceset="RESISTOR" device="0603" package3d_urn="urn:adsk.eagle:package:15661944/2" value="205"/>
+<part name="R10" library="LinnesLab-Passives" deviceset="RESISTOR" device="0603" package3d_urn="urn:adsk.eagle:package:15661944/2" value="205"/>
+<part name="R11" library="LinnesLab-Passives" deviceset="RESISTOR" device="0603" package3d_urn="urn:adsk.eagle:package:15661944/2" value="205"/>
+<part name="R12" library="LinnesLab-Passives" deviceset="RESISTOR" device="0603" package3d_urn="urn:adsk.eagle:package:15661944/2" value="10k"/>
+<part name="R13" library="LinnesLab-Passives" deviceset="RESISTOR" device="0603" package3d_urn="urn:adsk.eagle:package:15661944/2" value="10k"/>
+<part name="R14" library="LinnesLab-Passives" deviceset="RESISTOR" device="0603" package3d_urn="urn:adsk.eagle:package:15661944/2" value="10k"/>
 <part name="SUPPLY11" library="LinnesLab-Symbols" deviceset="3.3V" device=""/>
 <part name="SUPPLY12" library="LinnesLab-Symbols" deviceset="3.3V" device=""/>

Commit message: Changes
Parts:
- R2: value (none) -> 4.7k
Changed lines of the file:
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@@
 <part name="LDO1" library="LinnesLab-Power" deviceset="MIC550X" device="" package3d_urn="urn:adsk.eagle:package:15662427/2"/>
 <part name="U1" library="LinnesLab-Power" deviceset="MCP73831" device=".SOT23-5" package3d_urn="urn:adsk.eagle:package:18172171/2"/>
-<part name="R2" library="LinnesLab-Passives" deviceset="RESISTOR" device="0603" package3d_urn="urn:adsk.eagle:package:15661944/2"/>
+<part name="R2" library="LinnesLab-Passives" deviceset="RESISTOR" device="0603" package3d_urn="urn:adsk.eagle:package:15661944/2" value="4.7k"/>
 <part name="R3" library="LinnesLab-Passives" deviceset="RESISTOR" device="0603" package3d_urn="urn:adsk.eagle:package:15661944/2" value="100k"/>
 <part name="SW2" library="LinnesLab-Switches" deviceset="SWITCH.JS202011JXQN" device="UPWARDS"/>

Commit message: orlando made changes and ordered boards
Parts:
- C1, C2: value 22p -> 0.1u
- C3: value 0.1u -> 2.2u
- C4: value 2.2u -> 22p
- C5: value 0.1u -> 22p
- R2: value 4.7k -> 100k
- R3: value 100k -> 4.7k
- U1: value MCP73831.SOT23-5 -> ATMEGA328P_TQFP; device LinnesLab-Power:MCP73831.SOT23-5 -> LinnesLab-Microcontrollers:ATMEGA328P_TQFP
- U2: value ATMEGA328P_TQFP -> MCP73831.SOT23-5; device LinnesLab-Microcontrollers:ATMEGA328P_TQFP -> LinnesLab-Power:MCP73831.SOT23-5
Connections:
- removed net N$1: C3.2, R1.1, U2.PC6(/RESET)
- net 3.3V: now also C1.1, C3.1, U1.AVCC, U1.VCC@4, U1.VCC@6; no longer C4.1, C5.1, U2.AVCC, U2.VCC@4, U2.VCC@6
- net ACTION: now also R13.2, SW4.B, U1.ADC6; no longer R14.2, SW5.B, U2.ADC6
- net CHRG.STAT: now also R2.1; no longer R3.1
- net DTR: now also C2.1
- net GND: now also C3.2, R3.1, U1.AGND, U1.GND@3, U1.GND@5, U2.VSS; no longer C2.2, R2.1, U1.VSS, U2.AGND, U2.GND@3, U2.GND@5
- net LD1: now also U1.D4/PD4(XCK/T0); no longer U2.D4/PD4(XCK/T0)
- net LD10: now also U1.D12/PB4(MISO); no longer U2.D12/PB4(MISO)
- net LD11: now also U1.D11/PB3(MOSI/OC2); no longer U2.D11/PB3(MOSI/OC2)
- net LD12: now also U1.D10/PB2(SS/OC1B); no longer U2.D10/PB2(SS/OC1B)
- net LD13: now also U1.D9/PB1(OC1A); no longer U2.D9/PB1(OC1A)
- net LD14: now also U1.D8/PB0(ICP); no longer U2.D8/PB0(ICP)
- net LD15: now also U1.D7/PD7(AIN1); no longer U2.D7/PD7(AIN1)
- net LD16: now also U1.D6/PD6(AIN0); no longer U2.D6/PD6(AIN0)
- net LD2: now also U1.D3/PD3(INT1); no longer U2.D3/PD3(INT1)
- net LD3: now also U1.D2/PD2(INT0); no longer U2.D2/PD2(INT0)
- net LD4: now also U1.PC5(ADC5/SCL); no longer U2.PC5(ADC5/SCL)
- net LD5: now also U1.PC4(ADC4/SDA); no longer U2.PC4(ADC4/SDA)
- net LD6: now also U1.PC3(ADC3); no longer U2.PC3(ADC3)
- net LD7: now also U1.PC2(ADC2); no longer U2.PC2(ADC2)
- net LD8: now also U1.PC1(ADC1); no longer U2.PC1(ADC1)
- net LD9: now also U1.D13/PB5(SCK); no longer U2.D13/PB5(SCK)
- net LEFT: now also U1.PC0(ADC0); no longer U2.PC0(ADC0)
- net MODE: now also U1.D5/PD5(T1); no longer U2.D5/PD5(T1)
- net N$3: now also C4.1, U1.PB6(XTAL1/TOSC1); no longer C2.1, U2.PB6(XTAL1/TOSC1)
- net N$4: now also C5.1, U1.PB7(XTAL2/TOSC2); no longer C1.1, U2.PB7(XTAL2/TOSC2)
- net N$6: now also U2.STAT; no longer U1.STAT
- net N$60: now also D1.A; no longer D2.A
- net N$64: now also R3.2, U2.PROG; no longer R2.2, U1.PROG
- net RESET: now also C2.2, R1.1, U1.PC6(/RESET); no longer C3.1
- net RIGHT: now also R14.2, SW5.B, U1.ADC7; no longer R13.2, SW4.B, U2.ADC7
- net RXD: now also U1.D0/PD0(RXD); no longer U2.D0/PD0(RXD)
- net TXD: now also U1.D1/PD1(TXD); no longer U2.D1/PD1(TXD)
- net VIN: now also C6.1, R2.2, U2.VIN; no longer C9.1, R3.2, U1.VIN
- net VLIPO: now also C9.1, U2.VBAT; no longer C6.1, U1.VBAT
- net V_USB: now also D2.A; no longer D1.A
Other:
- moved on the sheet: C1, C2, C3, C4, C5, C6, C9, D1, D2, R13, R14, R2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
